Commit message: Clean up some non-conforming URDF elements
In anticipation of schema checking for URDF, clean up some structure
errors in robotiq models.

* The `cable` element does not obey drake namespace style for
  extensions, and has not had code support since removal of matlab files
  in 2017.
* Move some `inertial` elements to their likely intended homes.

File: atlas/robotiq.urdf (robot description, URDF)
Before this commit: robot s-model_articulated, 34 links, 33 joints
Links:
- link palm: mass None -> 1.3

File: atlas/robotiq_simple.urdf (robot description, URDF)
Before this commit: robot s-model_articulated, 13 links, 12 joints
Links:
- link palm: mass None -> 1.3

File: atlas/robotiq_tendons.urdf (robot description, URDF)
Before this commit: robot s-model_articulated, 14 links, 13 joints
Links:
- link palm: mass None -> 1.3
