Commit message: [atlas] Convert obj2gltf on visual meshes

File: atlas/atlas_convex_hull.urdf (robot description, URDF)
Before this commit: robot atlas, 70 links, 69 joints
Links:
- link l_clav: geometry collision mesh filename=package://drake_models/atlas/meshes/r_clav_chull.obj; visual mesh filename=package://drake_models/atlas/meshes/r_clav.gltf
- link l_foot: geometry collision mesh filename=package://drake_models/atlas/meshes/l_foot_chull.obj; collision sphere radius=0.0
- link l_larm: geometry collision mesh filename=package://drake_models/atlas/meshes/r_larm_chull.obj; visual mesh filename=package://drake_models/atlas/meshes/r_larm.gltf
- link l_lfarm: geometry collision mesh filename=package://drake_models/atlas/meshes/r_hand_chull.obj; visual mesh filename=package://drake_models/atlas/meshes/r_hand.gltf
- link l_lglut: geometry collision mesh filename=package://drake_models/atlas/meshes/l_lglut_chull.obj; visual mesh filename=package://drake_models/atlas/meshes/l_lglut.gltf
- link l_lleg: geometry collision mesh filename=package://drake_models/atlas/meshes/l_lleg_chull.obj; visual mesh filename=package://drake_models/atlas/meshes/l_lleg.gltf
- link l_scap: geometry collision mesh filename=package://drake_models/atlas/meshes/r_scap_chull.obj; visual mesh filename=package://drake_models/atlas/meshes/r_scap.gltf
- link l_talus: geometry visual mesh filename=package://drake_models/atlas/meshes/l_talus.gltf
- link l_uarm: geometry collision mesh filename=package://drake_models/atlas/meshes/r_uarm_chull.obj; visual mesh filename=package://drake_models/atlas/meshes/r_uarm.gltf
- link l_ufarm: geometry collision mesh filename=package://drake_models/atlas/meshes/r_farm_chull.obj; visual mesh filename=package://drake_models/atlas/meshes/r_farm.gltf
- link l_uglut: geometry collision mesh filename=package://drake_models/atlas/meshes/l_uglut_chull.obj; visual mesh filename=package://drake_models/atlas/meshes/l_uglut.gltf
- link l_uleg: geometry collision mesh filename=package://drake_models/atlas/meshes/l_uleg_chull.obj; visual mesh filename=package://drake_models/atlas/meshes/l_uleg.gltf
- link ltorso: geometry visual mesh filename=package://drake_models/atlas/meshes/ltorso.gltf
- link mtorso: geometry visual mesh filename=package://drake_models/atlas/meshes/mtorso.gltf
- link pelvis: geometry collision mesh filename=package://drake_models/atlas/meshes/pelvis_chull.obj; visual mesh filename=package://drake_models/atlas/meshes/pelvis.gltf
- link r_clav: geometry collision mesh filename=package://drake_models/atlas/meshes/r_clav_chull.obj; visual mesh filename=package://drake_models/atlas/meshes/r_clav.gltf
- link r_foot: geometry collision mesh filename=package://drake_models/atlas/meshes/r_foot_chull.obj; collision sphere radius=0.0
- link r_larm: geometry collision mesh filename=package://drake_models/atlas/meshes/r_larm_chull.obj; visual mesh filename=package://drake_models/atlas/meshes/r_larm.gltf
- link r_lfarm: geometry collision mesh filename=package://drake_models/atlas/meshes/r_hand_chull.obj; visual mesh filename=package://drake_models/atlas/meshes/r_hand.gltf
- link r_lglut: geometry collision mesh filename=package://drake_models/atlas/meshes/r_lglut_chull.obj; visual mesh filename=package://drake_models/atlas/meshes/r_lglut.gltf
- link r_lleg: geometry collision mesh filename=package://drake_models/atlas/meshes/r_lleg_chull.obj; visual mesh filename=package://drake_models/atlas/meshes/r_lleg.gltf
- link r_scap: geometry collision mesh filename=package://drake_models/atlas/meshes/r_scap_chull.obj; visual mesh filename=package://drake_models/atlas/meshes/r_scap.gltf
- link r_talus: geometry visual mesh filename=package://drake_models/atlas/meshes/r_talus.gltf
- link r_uarm: geometry collision mesh filename=package://drake_models/atlas/meshes/r_uarm_chull.obj; visual mesh filename=package://drake_models/atlas/meshes/r_uarm.gltf
- link r_ufarm: geometry collision mesh filename=package://drake_models/atlas/meshes/r_farm_chull.obj; visual mesh filename=package://drake_models/atlas/meshes/r_farm.gltf
- link r_uglut: geometry collision mesh filename=package://drake_models/atlas/meshes/r_uglut_chull.obj; visual mesh filename=package://drake_models/atlas/meshes/r_uglut.gltf
- link r_uleg: geometry collision mesh filename=package://drake_models/atlas/meshes/r_uleg_chull.obj; visual mesh filename=package://drake_models/atlas/meshes/r_uleg.gltf
- link utorso: geometry collision mesh filename=package://drake_models/atlas/meshes/utorso_chull.obj; visual mesh filename=package://drake_models/atlas/meshes/utorso.gltf

File: atlas/atlas_minimal_contact.urdf (robot description, URDF)
Before this commit: robot atlas, 60 links, 59 joints
Links:
- link head: geometry visual mesh filename=package://drake_models/atlas/meshes/head.gltf
- link hokuyo_link: geometry visual mesh filename=package://drake_models/atlas/meshes/head_camera.gltf
- link l_clav: geometry visual mesh filename=package://drake_models/atlas/meshes/r_clav.gltf
- link l_foot: geometry collision sphere radius=0.0; collision sphere radius=0.0
- link l_larm: geometry visual mesh filename=package://drake_models/atlas/meshes/r_larm.gltf
- link l_lfarm: geometry visual mesh filename=package://drake_models/atlas/meshes/r_hand.gltf
- link l_lglut: geometry visual mesh filename=package://drake_models/atlas/meshes/l_lglut.gltf
- link l_lleg: geometry visual mesh filename=package://drake_models/atlas/meshes/l_lleg.gltf
- link l_scap: geometry visual mesh filename=package://drake_models/atlas/meshes/r_scap.gltf
- link l_talus: geometry visual mesh filename=package://drake_models/atlas/meshes/l_talus.gltf
- link l_uarm: geometry visual mesh filename=package://drake_models/atlas/meshes/r_uarm.gltf
- link l_ufarm: geometry visual mesh filename=package://drake_models/atlas/meshes/r_farm.gltf
- link l_uglut: geometry visual mesh filename=package://drake_models/atlas/meshes/l_uglut.gltf
- link l_uleg: geometry visual mesh filename=package://drake_models/atlas/meshes/l_uleg.gltf
- link ltorso: geometry visual mesh filename=package://drake_models/atlas/meshes/ltorso.gltf
- link mtorso: geometry visual mesh filename=package://drake_models/atlas/meshes/mtorso.gltf
- link pelvis: geometry visual mesh filename=package://drake_models/atlas/meshes/pelvis.gltf
- link r_clav: geometry visual mesh filename=package://drake_models/atlas/meshes/r_clav.gltf
- link r_foot: geometry collision sphere radius=0.0; collision sphere radius=0.0
- link r_larm: geometry visual mesh filename=package://drake_models/atlas/meshes/r_larm.gltf
- link r_lfarm: geometry visual mesh filename=package://drake_models/atlas/meshes/r_hand.gltf
- link r_lglut: geometry visual mesh filename=package://drake_models/atlas/meshes/r_lglut.gltf
- link r_lleg: geometry visual mesh filename=package://drake_models/atlas/meshes/r_lleg.gltf
- link r_scap: geometry visual mesh filename=package://drake_models/atlas/meshes/r_scap.gltf
- link r_talus: geometry visual mesh filename=package://drake_models/atlas/meshes/r_talus.gltf
- link r_uarm: geometry visual mesh filename=package://drake_models/atlas/meshes/r_uarm.gltf
- link r_ufarm: geometry visual mesh filename=package://drake_models/atlas/meshes/r_farm.gltf
- link r_uglut: geometry visual mesh filename=package://drake_models/atlas/meshes/r_uglut.gltf
- link r_uleg: geometry visual mesh filename=package://drake_models/atlas/meshes/r_uleg.gltf
- link utorso: geometry visual mesh filename=package://drake_models/atlas/meshes/utorso.gltf

Commit message: Fixing normals

File: atlas/atlas_convex_hull.urdf (robot description, URDF)
Before this commit: robot atlas, 70 links, 69 joints
Links:
- link head: geometry collision mesh filename=package://drake_models/atlas/meshes/head_chull.obj; visual mesh filename=package://drake_models/atlas/meshes/head.gltf
- link hokuyo_link: geometry collision mesh filename=package://drake_models/atlas/meshes/head_camera_chull.obj; visual mesh filename=package://drake_models/atlas/meshes/head_camera.gltf
- link left_palm: geometry collision mesh filename=package://drake_models/atlas/meshes/GRIPPER_OPEN_chull.obj scale=1 1 1; visual mesh filename=package://drake_models/atlas/meshes/GRIPPER_OPEN_chull.gltf scale=1 1 1
- link right_palm: geometry collision mesh filename=package://drake_models/atlas/meshes/GRIPPER_OPEN_chull.obj scale=1 1 1; visual mesh filename=package://drake_models/atlas/meshes/GRIPPER_OPEN_chull.gltf scale=1 1 1
