Commit message: [tri_homecart] Convert visual meshes to glTF

File: tri_homecart/homecart_bimanual.urdf.xacro (robot description, xacro)
@@ -47,5 +47,5 @@
                 rpy="0 0 0"/>
         <geometry>
-          <mesh filename="package://drake_models/tri_homecart/assets/homecart_arm_mount_stack.obj"/>
+          <mesh filename="package://drake_models/tri_homecart/assets/homecart_arm_mount_stack.gltf"/>
         </geometry>
       </visual>
@@ -58,5 +58,5 @@
         <origin xyz="0 0 0.0" rpy="0 0 0"/>
         <geometry>
-          <mesh filename="package://drake_models/tri_homecart/assets/homecart_arm_mount_cantilever.obj"/>
+          <mesh filename="package://drake_models/tri_homecart/assets/homecart_arm_mount_cantilever.gltf"/>
         </geometry>
       </visual>
@@ -147,5 +147,5 @@
       <origin xyz="0 0 0.0" rpy="0 0 0"/>
       <geometry>
-        <mesh filename="package://drake_models/tri_homecart/assets/homecart_baseplate.obj"/>
+        <mesh filename="package://drake_models/tri_homecart/assets/homecart_baseplate.gltf"/>
       </geometry>
     </visual>
@@ -172,5 +172,5 @@
       <origin xyz="0 0 0.0" rpy="0 0 0"/>
       <geometry>
-        <mesh filename="package://drake_models/tri_homecart/assets/homecart_basecart.obj"/>
+        <mesh filename="package://drake_models/tri_homecart/assets/homecart_basecart.gltf"/>
       </geometry>
     </visual>
@@ -224,5 +224,5 @@
     <origin xyz="0 0 0" rpy="0 0 0"/>
       <geometry>
-        <mesh filename="package://drake_models/tri_homecart/assets/homecart_bimanual_upper_structure.obj"/>
+        <mesh filename="package://drake_models/tri_homecart/assets/homecart_bimanual_upper_structure.gltf"/>
       </geometry>
     </visual>

File: tri_homecart/homecart_cutting_board.sdf.xacro (robot description, xacro)
@@ -38,5 +38,5 @@
         <geometry>
           <mesh>
-            <uri>package://drake_models/tri_homecart/assets/homecart_cutting_board.obj</uri>
+            <uri>package://drake_models/tri_homecart/assets/homecart_cutting_board.gltf</uri>
             <scale>1.0 1.0 1.0</scale>
           </mesh>

Commit message: [homecart] URDF text cleanups
These files escaped a previous cleanup pass in drake by hiding in
models.

File: tri_homecart/homecart_bimanual.urdf.xacro (robot description, xacro)
@@ -25,7 +25,5 @@
       respect to the robot arm origins.
   -->
-  <link name="homecart_base_link">
-    <origin xyz="0 0 0" rpy="0 0 0"/>
-  </link>
+  <link name="homecart_base_link"/>
   <xacro:property name="arm_mount_cantilever_length" value="0.254"/>
   <xacro:property name="arm_mount_cantilever_height" value="0.015"/>
@@ -105,7 +103,5 @@
       <child link="${side}arm_mount_stack_link"/>
     </joint>
-    <link name="${side}arm_base_link">
-      <origin xyz="0 0 0" rpy="0 0 0"/>
-    </link>
+    <link name="${side}arm_base_link"/>
     <joint name="${side}arm_base_joint" type="fixed">
       <origin xyz="0 0 ${num_plates*0.02}" rpy="0 0 0"/>
