Commit message: [jaco_description] Convert obj2gltf on meshes
After conversion, the following additional steps were taken

1. Tweak glTF materials to more closely reflect the
   rendered appearance of the original OBJs.
2. Fixed extensive normals issues (the glTFs had normals,
   but they were *bad*).
3. Removal of `<material>` tags in the urdf files.
4. Removal of visual-only and unused .obj files.
   - Note: some objs were converted, but are unreferenced.

File: jaco_description/urdf/j2n6s300.urdf (robot description, URDF)
Before this commit: robot j2n6s300, 15 links, 14 joints
Links:
- link j2n6s300_link_1: geometry collision cylinder length=0.06 radius=0.025; visual mesh filename=package://drake_models/jaco_description/meshes/ring_big.gltf
- link j2n6s300_link_2: geometry collision cylinder length=0.3 radius=0.025; visual mesh filename=package://drake_models/jaco_description/meshes/arm.gltf
- link j2n6s300_link_3: geometry collision cylinder length=0.17 radius=0.025; visual mesh filename=package://drake_models/jaco_description/meshes/forearm.gltf
- link j2n6s300_link_4: geometry collision cylinder length=0.01 radius=0.025; visual mesh filename=package://drake_models/jaco_description/meshes/ring_small.g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
- link j2n6s300_link_5: geometry collision cylinder length=0.01 radius=0.025; visual mesh filename=package://drake_models/jaco_description/meshes/ring_small.g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
- link j2n6s300_link_6: geometry collision cylinder length=0.01 radius=0.025; visual mesh filename=package://drake_models/jaco_description/meshes/hand_3finger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
- link j2n6s300_link_base: geometry collision cylinder length=0.075 radius=0.025; visual mesh filename=package://drake_models/jaco_description/meshes/base.gltf

File: jaco_description/urdf/j2s7s300.urdf (robot description, URDF)
Before this commit: robot j2s7s300, 16 links, 15 joints
Links:
- link j2s7s300_link_1: geometry collision mesh filename=package://drake_models/jaco_description/meshes/shoulder.gltf; visual mesh filename=package://drake_models/jaco_description/meshes/ring_big.gltf
- link j2s7s300_link_2: geometry collision mesh filename=package://drake_models/jaco_description/meshes/arm_half_1.g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; visual mesh filename=package://drake_models/jaco_description/meshes/arm_half_1.g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
- link j2s7s300_link_3: geometry collision mesh filename=package://drake_models/jaco_description/meshes/arm_half_2.g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; visual mesh filename=package://drake_models/jaco_description/meshes/arm_half_2.g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
- link j2s7s300_link_4: geometry collision mesh filename=package://drake_models/jaco_description/meshes/forearm.gltf; visual mesh filename=package://drake_models/jaco_description/meshes/forearm.gltf
- link j2s7s300_link_5: geometry collision mesh filename=package://drake_models/jaco_description/meshes/wrist_spheri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; visual mesh filename=package://drake_models/jaco_description/meshes/ring_small.g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
- link j2s7s300_link_6: geometry collision mesh filename=package://drake_models/jaco_description/meshes/wrist_spheri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; visual mesh filename=package://drake_models/jaco_description/meshes/ring_small.g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
- link j2s7s300_link_7: geometry collision mesh filename=package://drake_models/jaco_description/meshes/hand_3finger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; visual mesh filename=package://drake_models/jaco_description/meshes/hand_3finger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
- link j2s7s300_link_base: geometry collision mesh filename=package://drake_models/jaco_description/meshes/base.gltf; visual mesh filename=package://drake_models/jaco_description/meshes/base.gltf

File: jaco_description/urdf/j2s7s300_arm.urdf (robot description, URDF)
Before this commit: robot j2s7s300_arm, 9 links, 8 joints
Links:
- link j2s7s300_link_1: geometry collision mesh filename=package://drake_models/jaco_description/meshes/shoulder.obj; visual mesh filename=package://drake_models/jaco_description/meshes/ring_big.gltf
- link j2s7s300_link_2: geometry collision mesh filename=package://drake_models/jaco_description/meshes/arm_half_1.o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; visual mesh filename=package://drake_models/jaco_description/meshes/arm_half_1.g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
- link j2s7s300_link_3: geometry collision mesh filename=package://drake_models/jaco_description/meshes/arm_half_2.o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; visual mesh filename=package://drake_models/jaco_description/meshes/arm_half_2.g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
- link j2s7s300_link_4: geometry collision mesh filename=package://drake_models/jaco_description/meshes/forearm.obj; visual mesh filename=package://drake_models/jaco_description/meshes/forearm.gltf
- link j2s7s300_link_5: geometry collision mesh filename=package://drake_models/jaco_description/meshes/wrist_spheri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; visual mesh filename=package://drake_models/jaco_description/meshes/ring_small.g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
- link j2s7s300_link_6: geometry collision mesh filename=package://drake_models/jaco_description/meshes/wrist_spheri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; visual mesh filename=package://drake_models/jaco_description/meshes/ring_small.g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
- link j2s7s300_link_base: geometry collision mesh filename=package://drake_models/jaco_description/meshes/base.obj; visual mesh filename=package://drake_models/jaco_description/meshes/base.gltf

File: jaco_description/urdf/j2s7s300_arm_sphere_collision.urdf (robot description, URDF)
Before this commit: robot j2s7s300_arm, 9 links, 8 joints
Links:
- link j2s7s300_link_1: geometry collision sphere radius=0.02; collision sphere radius=0.02
- link j2s7s300_link_2: geometry collision sphere radius=0.02; collision sphere radius=0.02
- link j2s7s300_link_3: geometry collision sphere radius=0.015; collision sphere radius=0.015
- link j2s7s300_link_4: geometry collision sphere radius=0.015; collision sphere radius=0.015
- link j2s7s300_link_5: geometry collision sphere radius=0.0325; collision sphere radius=0.035
- link j2s7s300_link_6: geometry collision sphere radius=0.035; collision sphere radius=0.035
- link j2s7s300_link_base: geometry collision sphere radius=0.045; collision sphere radius=0.045

File: jaco_description/urdf/j2s7s300_hand.urdf (robot description, URDF)
Before this commit: robot j2s7s300_hand, 8 links, 7 joints
Links:
- link hand_base: geometry collision mesh filename=package://drake_models/jaco_description/meshes/hand_3finger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; visual mesh filename=package://drake_models/jaco_description/meshes/hand_3finger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

File: jaco_description/urdf/j2s7s300_hand_sphere_collision.urdf (robot description, URDF)
Before this commit: robot j2s7s300_hand, 8 links, 7 joints
Links:
- link hand_base: geometry collision sphere radius=0.03; collision sphere radius=0.03

File: jaco_description/urdf/j2s7s300_sphere_collision.urdf (robot description, URDF)
Before this commit: robot j2s7s300, 16 links, 15 joints
Links:
- link j2s7s300_link_1: geometry collision sphere radius=0.02; collision sphere radius=0.02
- link j2s7s300_link_2: geometry collision sphere radius=0.02; collision sphere radius=0.02
- link j2s7s300_link_3: geometry collision sphere radius=0.015; collision sphere radius=0.015
- link j2s7s300_link_4: geometry collision sphere radius=0.015; collision sphere radius=0.015
- link j2s7s300_link_5: geometry collision sphere radius=0.0325; collision sphere radius=0.035
- link j2s7s300_link_6: geometry collision sphere radius=0.035; collision sphere radius=0.035
- link j2s7s300_link_7: geometry collision sphere radius=0.03; collision sphere radius=0.03
- link j2s7s300_link_base: geometry collision sphere radius=0.045; collision sphere radius=0.045
