Commit message: [skydio_2] Converg obj2gltf for visual meshes

File: skydio_2/quadrotor.urdf (robot description, URDF)
Before this commit: robot quadrotor, 1 links, 0 joints
Links:
- link base_link: geometry collision box size=.36 .4 .06; visual mesh filename=package://drake_models/skydio_2/skydio_2_1000_poly.gltf scale=.00254
