Commit message: [realsense2] Convert obj2gltf visual models
- Update the xacro files (we no longer should apply a material to the glTF).
- Update the path to the geometry to use the drake_models package.
- Update swapping stl -> gltf.

File: realsense2_description/urdf/_d415.urdf.xacro (robot description, xacro)
@@ -21,5 +21,4 @@
 <robot name="sensor_d415" xmlns:xacro="http://ros.org/wiki/xacro">
   <!-- Includes -->
-  <xacro:include filename="$(find realsense2_description)/urdf/_materials.urdf.xacro" />
   <xacro:include filename="$(find realsense2_description)/urdf/_usb_plug.urdf.xacro" />
   <xacro:macro name="sensor_d415" params="parent *origin  name:=camera  use_nominal_extrinsics:=false add_plug:=false use_mesh:=true">
@@ -61,5 +60,4 @@
             <mesh filename="file://$(find realsense2_description)/meshes/d415.stl" />
           </geometry>
-          <material name="aluminum"/>
         </xacro:if>
         <xacro:unless value="${use_mesh}">

File: realsense2_description/urdf/d415.urdf (robot description, URDF)
Before this commit: robot realsense2_camera, 3 links, 2 joints
Links:
- link camera_link: geometry collision box size=0.02005 0.099 0.023; visual mesh filename=package://drake_models/realsense2_description/meshes/d415.g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
