Commit message: [ur_description] Update to new mesh paths

File: ur_description/urdf/ur3e.urdf.xacro (robot description, xacro)
@@ -71,5 +71,5 @@
         <origin rpy="0 0 0" xyz="0.0 0.0 0.0"/>
         <geometry>
-          <mesh filename="package://drake_models/ur3e/base.obj"/>
+          <mesh filename="package://drake_models/ur_description/meshes/base.obj"/>
         </geometry>
         <material name="LightGrey">
@@ -148,5 +148,5 @@
         <origin rpy="0 0 0" xyz="0.0 0.0 0.0"/>
         <geometry>
-          <mesh filename="package://drake_models/ur3e/shoulder.obj"/>
+          <mesh filename="package://drake_models/ur_description/meshes/shoulder.obj"/>
         </geometry>
         <material name="LightGrey">
@@ -209,5 +209,5 @@
         <origin rpy="0 0 0" xyz="0.0 0.0 0.0"/>
         <geometry>
-          <mesh filename="package://drake_models/ur3e/upperarm.obj"/>
+          <mesh filename="package://drake_models/ur_description/meshes/upperarm.obj"/>
         </geometry>
         <material name="LightGrey">
@@ -324,5 +324,5 @@
         <origin rpy="0 0 0" xyz="0.0 0.0 0.0"/>
         <geometry>
-          <mesh filename="package://drake_models/ur3e/forearm.obj"/>
+          <mesh filename="package://drake_models/ur_description/meshes/forearm.obj"/>
         </geometry>
         <material name="LightGrey">
@@ -457,5 +457,5 @@
         <origin rpy="0 0 0" xyz="0.0 0.0 0.0"/>
         <geometry>
-          <mesh filename="package://drake_models/ur3e/wrist1.obj"/>
+          <mesh filename="package://drake_models/ur_description/meshes/wrist1.obj"/>
         </geometry>
         <material name="LightGrey">
@@ -530,5 +530,5 @@
         <origin rpy="0 0 0" xyz="0.0 0.0 0.0"/>
         <geometry>
-          <mesh filename="package://drake_models/ur3e/wrist2.obj"/>
+          <mesh filename="package://drake_models/ur_description/meshes/wrist2.obj"/>
         </geometry>
         <material name="LightGrey">
@@ -603,5 +603,5 @@
         <origin rpy="0 0 0" xyz="0.0 0.0 0.0"/>
         <geometry>
-          <mesh filename="package://drake_models/ur3e/wrist3.obj"/>
+          <mesh filename="package://drake_models/ur_description/meshes/wrist3.obj"/>
         </geometry>
         <material name="LightGrey">

File: ur_description/urdf/ur3e_cylinders_collision.urdf (robot description, URDF)
Before this commit: robot ur3e, 10 links, 9 joints
Links:
- link ur_base_link: geometry collision sphere radius=0.03; collision sphere radius=0.07
- link ur_forearm_link: geometry collision cylinder length=0.14 radius=0.034; collision cylinder length=0.185 radius=0.034
- link ur_shoulder_link: geometry collision cylinder length=0.16 radius=0.05; visual mesh filename=package://drake_models/ur_description/meshes/shoulder.obj
- link ur_upper_arm_link: geometry collision cylinder length=0.051 radius=0.05; collision cylinder length=0.11 radius=0.041
- link ur_wrist_1_link: geometry collision cylinder length=0.12 radius=0.034; visual mesh filename=package://drake_models/ur_description/meshes/wrist1.obj
- link ur_wrist_2_link: geometry collision cylinder length=0.092 radius=0.034; visual mesh filename=package://drake_models/ur_description/meshes/wrist2.obj
- link ur_wrist_3_link: geometry collision cylinder length=0.05 radius=0.034; visual mesh filename=package://drake_models/ur_description/meshes/wrist3.obj

File: ur_description/urdf/ur3e_spheres_collision.urdf (robot description, URDF)
Before this commit: robot ur3e, 10 links, 9 joints
Links:
- link ur_base_link: geometry collision sphere radius=0.03; collision sphere radius=0.055
- link ur_forearm_link: geometry collision sphere radius=0.03; collision sphere radius=0.03
- link ur_shoulder_link: geometry collision sphere radius=0.0525; collision sphere radius=0.0525
- link ur_upper_arm_link: geometry collision sphere radius=0.04; collision sphere radius=0.04
- link ur_wrist_1_link: geometry collision sphere radius=0.0375; collision sphere radius=0.0375
- link ur_wrist_2_link: geometry collision sphere radius=0.0375; collision sphere radius=0.0375
- link ur_wrist_3_link: geometry collision sphere radius=0.02; visual mesh filename=package://drake_models/ur_description/meshes/wrist3.obj

Commit message: [ur_description] Convert obj2gltf on visual meshes
This includes png->ktx conversion.

The mechanical conversion wasn't enough. The model had a metallic/roughness
/ambient occlusion map. This has been wired up into the model.
Reduced underlying base color to 80% to limit the amount of light
saturation happening compared to the phong model

File: ur_description/urdf/ur3e.urdf.xacro (robot description, xacro)
@@ -71,9 +71,6 @@
         <origin rpy="0 0 0" xyz="0.0 0.0 0.0"/>
         <geometry>
-          <mesh filename="package://drake_models/ur_description/meshes/base.obj"/>
+          <mesh filename="package://drake_models/ur_description/meshes/base.gltf"/>
         </geometry>
-        <material name="LightGrey">
-          <color rgba="0.7 0.7 0.7 1.0"/>
-        </material>
       </visual>
       <xacro:if value="${sphere_only_collision_shapes}">
@@ -148,9 +145,6 @@
         <origin rpy="0 0 0" xyz="0.0 0.0 0.0"/>
         <geometry>
-          <mesh filename="package://drake_models/ur_description/meshes/shoulder.obj"/>
+          <mesh filename="package://drake_models/ur_description/meshes/shoulder.gltf"/>
         </geometry>
-        <material name="LightGrey">
-          <color rgba="0.7 0.7 0.7 1.0"/>
-        </material>
       </visual>
       <xacro:if value="${sphere_only_collision_shapes}">
@@ -209,9 +203,6 @@
         <origin rpy="0 0 0" xyz="0.0 0.0 0.0"/>
         <geometry>
-          <mesh filename="package://drake_models/ur_description/meshes/upperarm.obj"/>
+          <mesh filename="package://drake_models/ur_description/meshes/upperarm.gltf"/>
         </geometry>
-        <material name="LightGrey">
-          <color rgba="0.7 0.7 0.7 1.0"/>
-        </material>
       </visual>
       <xacro:if value="${sphere_only_collision_shapes}">
@@ -324,9 +315,6 @@
         <origin rpy="0 0 0" xyz="0.0 0.0 0.0"/>
         <geometry>
-          <mesh filename="package://drake_models/ur_description/meshes/forearm.obj"/>
+          <mesh filename="package://drake_models/ur_description/meshes/forearm.gltf"/>
         </geometry>
-        <material name="LightGrey">
-          <color rgba="0.7 0.7 0.7 1.0"/>
-        </material>
       </visual>
       <xacro:if value="${sphere_only_collision_shapes}">
@@ -457,9 +445,6 @@
         <origin rpy="0 0 0" xyz="0.0 0.0 0.0"/>
         <geometry>
-          <mesh filename="package://drake_models/ur_description/meshes/wrist1.obj"/>
+          <mesh filename="package://drake_models/ur_description/meshes/wrist1.gltf"/>
         </geometry>
-        <material name="LightGrey">
-          <color rgba="0.7 0.7 0.7 1.0"/>
-        </material>
       </visual>
       <xacro:if value="${sphere_only_collision_shapes}">
@@ -530,9 +515,6 @@
         <origin rpy="0 0 0" xyz="0.0 0.0 0.0"/>
         <geometry>
-          <mesh filename="package://drake_models/ur_description/meshes/wrist2.obj"/>
+          <mesh filename="package://drake_models/ur_description/meshes/wrist2.gltf"/>
         </geometry>
-        <material name="LightGrey">
-          <color rgba="0.7 0.7 0.7 1.0"/>
-        </material>
       </visual>
       <xacro:if value="${sphere_only_collision_shapes}">
@@ -603,9 +585,6 @@
         <origin rpy="0 0 0" xyz="0.0 0.0 0.0"/>
         <geometry>
-          <mesh filename="package://drake_models/ur_description/meshes/wrist3.obj"/>
+          <mesh filename="package://drake_models/ur_description/meshes/wrist3.gltf"/>
         </geometry>
-        <material name="LightGrey">
-          <color rgba="0.7 0.7 0.7 1.0"/>
-        </material>
       </visual>
       <xacro:if value="${sphere_only_collision_shapes}">

File: ur_description/urdf/ur3e_cylinders_collision.urdf (robot description, URDF)
Before this commit: robot ur3e, 10 links, 9 joints
Links:
- link ur_base_link: geometry collision sphere radius=0.03; collision sphere radius=0.07
- link ur_forearm_link: geometry collision cylinder length=0.14 radius=0.034; collision cylinder length=0.185 radius=0.034
- link ur_shoulder_link: geometry collision cylinder length=0.16 radius=0.05; visual mesh filename=package://drake_models/ur_description/meshes/shoulder.gltf
- link ur_upper_arm_link: geometry collision cylinder length=0.051 radius=0.05; collision cylinder length=0.11 radius=0.041
- link ur_wrist_1_link: geometry collision cylinder length=0.12 radius=0.034; visual mesh filename=package://drake_models/ur_description/meshes/wrist1.gltf
- link ur_wrist_2_link: geometry collision cylinder length=0.092 radius=0.034; visual mesh filename=package://drake_models/ur_description/meshes/wrist2.gltf
- link ur_wrist_3_link: geometry collision cylinder length=0.05 radius=0.034; visual mesh filename=package://drake_models/ur_description/meshes/wrist3.gltf

File: ur_description/urdf/ur3e_spheres_collision.urdf (robot description, URDF)
Before this commit: robot ur3e, 10 links, 9 joints
Links:
- link ur_base_link: geometry collision sphere radius=0.03; collision sphere radius=0.055
- link ur_forearm_link: geometry collision sphere radius=0.03; collision sphere radius=0.03
- link ur_shoulder_link: geometry collision sphere radius=0.0525; collision sphere radius=0.0525
- link ur_upper_arm_link: geometry collision sphere radius=0.04; collision sphere radius=0.04
- link ur_wrist_1_link: geometry collision sphere radius=0.0375; collision sphere radius=0.0375
- link ur_wrist_2_link: geometry collision sphere radius=0.0375; collision sphere radius=0.0375
- link ur_wrist_3_link: geometry collision sphere radius=0.02; visual mesh filename=package://drake_models/ur_description/meshes/wrist3.gltf

Commit message: [ur_description] Convert obj2gltf on visual meshes
The mechanical conversion wasn't enough. The model had a metallic/roughness
/ambient occlusion map. This has been wired up into the model.
Reduced underlying base color to 80% to limit the amount of light
saturation happening compared to the phong model

File: ur_description/urdf/ur3e.urdf.xacro (robot description, xacro)
@@ -71,5 +71,5 @@
         <origin rpy="0 0 0" xyz="0.0 0.0 0.0"/>
         <geometry>
-          <mesh filename="package://drake_models/ur_description/meshes/base.obj"/>
+          <mesh filename="package://drake_models/ur_description/meshes/base.gltf"/>
         </geometry>
         <material name="LightGrey">
@@ -148,5 +148,5 @@
         <origin rpy="0 0 0" xyz="0.0 0.0 0.0"/>
         <geometry>
-          <mesh filename="package://drake_models/ur_description/meshes/shoulder.obj"/>
+          <mesh filename="package://drake_models/ur_description/meshes/shoulder.gltf"/>
         </geometry>
         <material name="LightGrey">
@@ -209,5 +209,5 @@
         <origin rpy="0 0 0" xyz="0.0 0.0 0.0"/>
         <geometry>
-          <mesh filename="package://drake_models/ur_description/meshes/upperarm.obj"/>
+          <mesh filename="package://drake_models/ur_description/meshes/upperarm.gltf"/>
         </geometry>
         <material name="LightGrey">
@@ -324,5 +324,5 @@
         <origin rpy="0 0 0" xyz="0.0 0.0 0.0"/>
         <geometry>
-          <mesh filename="package://drake_models/ur_description/meshes/forearm.obj"/>
+          <mesh filename="package://drake_models/ur_description/meshes/forearm.gltf"/>
         </geometry>
         <material name="LightGrey">
@@ -457,5 +457,5 @@
         <origin rpy="0 0 0" xyz="0.0 0.0 0.0"/>
         <geometry>
-          <mesh filename="package://drake_models/ur_description/meshes/wrist1.obj"/>
+          <mesh filename="package://drake_models/ur_description/meshes/wrist1.gltf"/>
         </geometry>
         <material name="LightGrey">
@@ -530,5 +530,5 @@
         <origin rpy="0 0 0" xyz="0.0 0.0 0.0"/>
         <geometry>
-          <mesh filename="package://drake_models/ur_description/meshes/wrist2.obj"/>
+          <mesh filename="package://drake_models/ur_description/meshes/wrist2.gltf"/>
         </geometry>
         <material name="LightGrey">
@@ -603,5 +603,5 @@
         <origin rpy="0 0 0" xyz="0.0 0.0 0.0"/>
         <geometry>
-          <mesh filename="package://drake_models/ur_description/meshes/wrist3.obj"/>
+          <mesh filename="package://drake_models/ur_description/meshes/wrist3.gltf"/>
         </geometry>
         <material name="LightGrey">

File: ur_description/urdf/ur3e_cylinders_collision.urdf (robot description, URDF)
Before this commit: robot ur3e, 10 links, 9 joints
Links:
- link ur_base_link: geometry collision sphere radius=0.03; collision sphere radius=0.07
- link ur_forearm_link: geometry collision cylinder length=0.14 radius=0.034; collision cylinder length=0.185 radius=0.034
- link ur_shoulder_link: geometry collision cylinder length=0.16 radius=0.05; visual mesh filename=package://drake_models/ur_description/meshes/shoulder.gltf
- link ur_upper_arm_link: geometry collision cylinder length=0.051 radius=0.05; collision cylinder length=0.11 radius=0.041
- link ur_wrist_1_link: geometry collision cylinder length=0.12 radius=0.034; visual mesh filename=package://drake_models/ur_description/meshes/wrist1.gltf
- link ur_wrist_2_link: geometry collision cylinder length=0.092 radius=0.034; visual mesh filename=package://drake_models/ur_description/meshes/wrist2.gltf
- link ur_wrist_3_link: geometry collision cylinder length=0.05 radius=0.034; visual mesh filename=package://drake_models/ur_description/meshes/wrist3.gltf

File: ur_description/urdf/ur3e_spheres_collision.urdf (robot description, URDF)
Before this commit: robot ur3e, 10 links, 9 joints
Links:
- link ur_base_link: geometry collision sphere radius=0.03; collision sphere radius=0.055
- link ur_forearm_link: geometry collision sphere radius=0.03; collision sphere radius=0.03
- link ur_shoulder_link: geometry collision sphere radius=0.0525; collision sphere radius=0.0525
- link ur_upper_arm_link: geometry collision sphere radius=0.04; collision sphere radius=0.04
- link ur_wrist_1_link: geometry collision sphere radius=0.0375; collision sphere radius=0.0375
- link ur_wrist_2_link: geometry collision sphere radius=0.0375; collision sphere radius=0.0375
- link ur_wrist_3_link: geometry collision sphere radius=0.02; visual mesh filename=package://drake_models/ur_description/meshes/wrist3.gltf
