Commit message: [dishes] Convert obj2gltf for visual meshes
OBJs are left in place as they are used for collision.

Upgraded mesh URIs to be package://.

File: dishes/evo_bowl_compliant.urdf (robot description, URDF)
Before this commit: robot bowl, 1 links, 0 joints
Links:
- link bowl: geometry collision mesh filename=package://drake_models/dishes/assets/evo_bowl_fine44k.vtk; visual mesh filename=package://drake_models/dishes/assets/evo_bowl.gltf
