Commit message: Improve Panda arm/hand collision model and filters

File: franka_description/urdf/panda_arm.urdf (robot description, URDF)
Before this commit: robot panda, 9 links, 8 joints
Links:
- added link panda_link2_extra; collision sphere radius=0.15
- added link panda_link5_extra; collision sphere radius=0.075
Joints:
- added joint panda_joint2_extra: type fixed, parent panda_link2, child panda_link2_extra, origin xyz=0 0 0 rpy=0 0 0
- added joint panda_joint5_extra: type fixed, parent panda_link5, child panda_link5_extra, origin xyz=0 0 0 rpy=0 0 0

File: franka_description/urdf/panda_arm_hand.urdf (robot description, URDF)
Before this commit: robot panda, 12 links, 11 joints
Links:
- added link panda_link2_extra; collision sphere radius=0.15
- added link panda_link5_extra; collision sphere radius=0.075
Joints:
- added joint panda_joint2_extra: type fixed, parent panda_link2, child panda_link2_extra, origin xyz=0 0 0 rpy=0 0 0
- added joint panda_joint5_extra: type fixed, parent panda_link5, child panda_link5_extra, origin xyz=0 0 0 rpy=0 0 0

Commit message: Split panda_link5 into lower/upper sections and improve collision filtering

File: franka_description/urdf/panda_arm.urdf (robot description, URDF)
Before this commit: robot panda, 9 links, 8 joints
Links:
- removed link panda_link5
- added link panda_link5_lower, mass 2.74; collision sphere radius=0.035; collision sphere radius=0.035
- added link panda_link5_upper; collision sphere radius=0.035; collision sphere radius=0.05
Joints:
- added joint panda_joint5_lower_upper: type fixed, parent panda_link5_lower, child panda_link5_upper, origin xyz=0 0 0 rpy=0 0 0
- joint panda_joint5: child panda_link5 -> panda_link5_lower
- joint panda_joint6: parent panda_link5 -> panda_link5_upper

File: franka_description/urdf/panda_arm_hand.urdf (robot description, URDF)
Before this commit: robot panda, 12 links, 11 joints
Links:
- removed link panda_link5
- added link panda_link5_lower, mass 2.74; collision sphere radius=0.035; collision sphere radius=0.035
- added link panda_link5_upper; collision sphere radius=0.035; collision sphere radius=0.05
Joints:
- added joint panda_joint5_lower_upper: type fixed, parent panda_link5_lower, child panda_link5_upper, origin xyz=0 0 0 rpy=0 0 0
- joint panda_joint5: child panda_link5 -> panda_link5_lower
- joint panda_joint6: parent panda_link5 -> panda_link5_upper
