Commit message: Move split link5 into different filename
Revert the changes to panda_arm{,_hand}.urdf.
Insted, copy the changes to new files named link5split.

File: franka_description/urdf/panda_arm_hand.urdf (robot description, URDF)
Before this commit: robot panda, 13 links, 12 joints
Links:
- removed link panda_link5_lower
- removed link panda_link5_upper
- added link panda_link5, mass 2.74; collision sphere radius=0.035; collision sphere radius=0.035
Joints:
- removed joint panda_joint5_lower_upper
- joint panda_joint5: child panda_link5_lower -> panda_link5
- joint panda_joint6: parent panda_link5_upper -> panda_link5

File: franka_description/urdf/panda_arm_hand_link5split.urdf (robot description, URDF)
Before this commit: robot panda, 9 links, 8 joints
Links:
- removed link panda_link5
- added link panda_hand, mass 0.73; collision sphere radius=0.05; collision sphere radius=0.05
- added link panda_leftfinger, mass 0.1; collision sphere radius=0.012; collision sphere radius=0.012
- added link panda_link5_lower, mass 2.74; collision sphere radius=0.035; collision sphere radius=0.035
- added link panda_link5_upper; collision sphere radius=0.035; collision sphere radius=0.05
- added link panda_rightfinger, mass 0.1; collision sphere radius=0.012; collision sphere radius=0.012
Joints:
- added joint panda_finger_joint1: type prismatic, parent panda_hand, child panda_leftfinger, origin xyz=0 0 0.0584 rpy=0 0 0, axis 0 1 0, limit lower=0.0 upper=0.04 effort=20 velocity=0.2
- added joint panda_finger_joint2: type prismatic, parent panda_hand, child panda_rightfinger, origin xyz=0 0 0.0584 rpy=0 0 0, axis 0 -1 0, limit lower=0.0 upper=0.04 effort=20 velocity=0.2
- added joint panda_hand_joint: type fixed, parent panda_link8, child panda_hand, origin xyz=0 0 0 rpy=0 0 -0.785398163397
- added joint panda_joint5_lower_upper: type fixed, parent panda_link5_lower, child panda_link5_upper, origin xyz=0 0 0 rpy=0 0 0
- joint panda_joint5: child panda_link5 -> panda_link5_lower
- joint panda_joint6: parent panda_link5 -> panda_link5_upper
